File: AGB-E02-20/AGB-E02-20.sch (KiCad schematic (older format))
At the start: 11 parts, among them U0 CartBus, U1 MX23L12806-12C, U2 LE26FV10N1TS

Commit message: Update AGB-E02-20
AGB-E02-20 looks much more "OEM" now
Parts:
- added G1: Nintendo Logo, Custom:Nintendo-GBA-Logo, symbol Mechanical:MountingHole
- added Pad1, Pad2: MountingHole_Pad, Custom:Nintendo_3x3_GNDPad, symbol Mechanical:MountingHole_Pad
- added Pad3, Pad4: MountingHole_Pad, Custom:Nintendo_1x1_Pad, symbol Mechanical:MountingHole_Pad
- added PlatedHole1: MountingHole, Custom:TestPoint_Plated_Hole_D2.0mm, symbol Mechanical:MountingHole
- C1, C2, C3: footprint Capacitor_SMD:C_0402_1005Metric -> Custom:C_0402_AGB
- R1, R2, R3: footprint Resistor_SMD:R_0402_1005Metric -> Custom:R_0603_AGB
- R4: footprint Capacitor_SMD:C_0603_1608Metric -> Custom:C_0603_AGB
- R5: footprint Resistor_SMD:R_0402_1005Metric -> Custom:R_0402_AGB-Opt
- U0: footprint NintendoFootprints:CartBus -> Connector_GameBoy:GameBoy_GamePak_AGB-002_P1.50mm_Edge
Changed lines of the file:
@@
 EESchema Schematic File Version 4
-EELAYER 29 0
+EELAYER 30 0
 EELAYER END
 $Descr A4 11693 8268
@@
 F 0 "U0" H 9050 5602 50  0000 C CNN
 F 1 "CartBus" H 9050 5511 50  0000 C CNN
-F 2 "NintendoFootprints:CartBus" H 8100 5975 50  0001 C CNN
+F 2 "Connector_GameBoy:GameBoy_GamePak_AGB-002_P1.50mm_Edge" H 8100 5975 50  0001 C CNN
 F 3 "" H 8100 5975 50  0001 C CNN
 	1    8100 5975
@@
 F 0 "R1" V 7800 2750 50  0000 L CNN
 F 1 "NC" H 7870 2755 50  0001 L CNN
-F 2 "Resistor_SMD:R_0402_1005Metric" V 7730 2800 50  0001 C CNN
+F 2 "Custom:R_0603_AGB" V 7730 2800 50  0001 C CNN
 F 3 "~" H 7800 2800 50  0001 C CNN
 	1    7800 2800
@@
 F 0 "R2" V 7800 2650 50  0000 L CNN
 F 1 "NC" H 7870 2655 50  0001 L CNN
-F 2 "Resistor_SMD:R_0402_1005Metric" V 7730 2700 50  0001 C CNN
+F 2 "Custom:R_0603_AGB" V 7730 2700 50  0001 C CNN
 F 3 "~" H 7800 2700 50  0001 C CNN
 	1    7800 2700
@@
 F 0 "R3" V 7800 2550 50  0000 L CNN
 F 1 "NC" H 7870 2555 50  0001 L CNN
-F 2 "Resistor_SMD:R_0402_1005Metric" V 7730 2600 50  0001 C CNN
+F 2 "Custom:R_0603_AGB" V 7730 2600 50  0001 C CNN
 F 3 "~" H 7800 2600 50  0001 C CNN
 	1    7800 2600
@@
 F 0 "C3" V 7875 1925 50  0000 L CNN
 F 1 "C" H 7840 1930 50  0001 L CNN
-F 2 "Capacitor_SMD:C_0402_1005Metric" H 7763 1825 50  0001 C CNN
+F 2 "Custom:C_0402_AGB" H 7763 1825 50  0001 C CNN
 F 3 "~" H 7725 1975 50  0001 C CNN
 	1    7725 1975
@@
 F 0 "R5" V 6275 850 50  0000 C CNN
 F 1 "NC" V 6350 850 50  0000 C CNN
-F 2 "Resistor_SMD:R_0402_1005Metric" V 6280 850 50  0001 C CNN
+F 2 "Custom:R_0402_AGB-Opt" V 6280 850 50  0001 C CNN
 F 3 "~" H 6350 850 50  0001 C CNN
 	1    6350 850
@@
 F 0 "C2" H 6060 1750 50  0000 R CNN
 F 1 "C" H 6060 1795 50  0001 R CNN
-F 2 "Capacitor_SMD:C_0402_1005Metric" H 6213 1600 50  0001 C CNN
+F 2 "Custom:C_0402_AGB" H 6213 1600 50  0001 C CNN
 F 3 "~" H 6175 1750 50  0001 C CNN
 	1    6175 1750
@@
 F 0 "C1" H 3715 2321 50  0000 L CNN
 F 1 "C" H 3715 2230 50  0000 L CNN
-F 2 "Capacitor_SMD:C_0402_1005Metric" H 3638 2125 50  0001 C CNN
+F 2 "Custom:C_0402_AGB" H 3638 2125 50  0001 C CNN
 F 3 "~" H 3600 2275 50  0001 C CNN
 	1    3600 2275
@@
 F 0 "R4" V 3525 3000 50  0000 C CNN
 F 1 "Cap" V 3600 3000 50  0000 C CNN
-F 2 "Capacitor_SMD:C_0603_1608Metric" V 3530 3000 50  0001 C CNN
+F 2 "Custom:C_0603_AGB" V 3530 3000 50  0001 C CNN
 F 3 "~" H 3600 3000 50  0001 C CNN
 	1    3600 3000
@@
 Text GLabel 4450 1900 0    50   Input ~ 0
 D7
+$Comp
+L Mechanical:MountingHole PlatedHole1
+U 1 1 5F1CF176
+P 6675 3625
+F 0 "PlatedHole1" H 6775 3671 50  0000 L CNN
+F 1 "MountingHole" H 6775 3580 50  0000 L CNN
+F 2 "Custom:TestPoint_Plated_Hole_D2.0mm" H 6675 3625 50  0001 C CNN
+F 3 "~" H 6675 3625 50  0001 C CNN
+	1    6675 3625
+	1    0    0    -1
+$EndComp
+$Comp
+L Mechanical:MountingHole_Pad Pad1
+U 1 1 5F1D11A5
+P 6725 4125
+F 0 "Pad1" V 6679 4275 50  0000 L CNN
+F 1 "MountingHole_Pad" V 6770 4275 50  0000 L CNN
+F 2 "Custom:Nintendo_3x3_GNDPad" H 6725 4125 50  0001 C CNN
+F 3 "~" H 6725 4125 50  0001 C CNN
+	1    6725 4125
+	0    1    1    0
+$EndComp
+$Comp
+L Mechanical:MountingHole_Pad Pad2
+U 1 1 5F1D1E72
+P 6725 4325
+F 0 "Pad2" V 6679 4475 50  0000 L CNN
+F 1 "MountingHole_Pad" V 6770 4475 50  0000 L CNN
+F 2 "Custom:Nintendo_3x3_GNDPad" H 6725 4325 50  0001 C CNN
+F 3 "~" H 6725 4325 50  0001 C CNN
+	1    6725 4325
+	0    1    1    0
+$EndComp
+$Comp
+L Mechanical:MountingHole_Pad Pad3
+U 1 1 5F1D2265
+P 6725 4525
+F 0 "Pad3" V 6679 4675 50  0000 L CNN
+F 1 "MountingHole_Pad" V 6770 4675 50  0000 L CNN
+F 2 "Custom:Nintendo_1x1_Pad" H 6725 4525 50  0001 C CNN
+F 3 "~" H 6725 4525 50  0001 C CNN
+	1    6725 4525
+	0    1    1    0
+$EndComp
+$Comp
+L power:GND #PWR0134
+U 1 1 5F1D3C86
+P 6625 4125
+F 0 "#PWR0134" H 6625 3875 50  0001 C CNN
+F 1 "GND" V 6625 3900 50  0000 C CNN
+F 2 "" H 6625 4125 50  0001 C CNN
+F 3 "" H 6625 4125 50  0001 C CNN
+	1    6625 4125
+	0    1    1    0
+$EndComp
+$Comp
+L power:GND #PWR0135
+U 1 1 5F1D408B
+P 6625 4325
+F 0 "#PWR0135" H 6625 4075 50  0001 C CNN
+F 1 "GND" V 6625 4100 50  0000 C CNN
+F 2 "" H 6625 4325 50  0001 C CNN
+F 3 "" H 6625 4325 50  0001 C CNN
+	1    6625 4325
+	0    1    1    0
+$EndComp
+$Comp
+L power:GND #PWR0136
+U 1 1 5F1D4442
+P 6625 4525
+F 0 "#PWR0136" H 6625 4275 50  0001 C CNN
+F 1 "GND" V 6625 4300 50  0000 C CNN
+F 2 "" H 6625 4525 50  0001 C CNN
+F 3 "" H 6625 4525 50  0001 C CNN
+	1    6625 4525
+	0    1    1    0
+$EndComp
+$Comp
+L Mechanical:MountingHole G1
+U 1 1 5F1DA8DA
+P 6775 4925
+F 0 "G1" H 6875 4971 50  0000 L CNN
+F 1 "Nintendo Logo" H 6875 4880 50  0000 L CNN
+F 2 "Custom:Nintendo-GBA-Logo" H 6775 4925 50  0001 C CNN
+F 3 "~" H 6775 4925 50  0001 C CNN
+	1    6775 4925
+	1    0    0    -1
+$EndComp
+$Comp
+L Mechanical:MountingHole_Pad Pad4
+U 1 1 5F207589
+P 6725 4725
+F 0 "Pad4" V 6679 4875 50  0000 L CNN
+F 1 "MountingHole_Pad" V 6770 4875 50  0000 L CNN
+F 2 "Custom:Nintendo_1x1_Pad" H 6725 4725 50  0001 C CNN
+F 3 "~" H 6725 4725 50  0001 C CNN
+	1    6725 4725
+	0    1    1    0
+$EndComp
+$Comp
+L power:GND #PWR0137
+U 1 1 5F20758F
+P 6625 4725
+F 0 "#PWR0137" H 6625 4475 50  0001 C CNN
+F 1 "GND" V 6625 4500 50  0000 C CNN
+F 2 "" H 6625 4725 50  0001 C CNN
+F 3 "" H 6625 4725 50  0001 C CNN
+	1    6625 4725
+	0    1    1    0
+$EndComp
 $EndSCHEMATC

Commit message: Update AGB-E02-20
AGB-E02-20 is now mostly identical to the original pcb (this was a lot of work)
Parts:
- C1, C2, C3: symbol Device:C -> AGB-E02-20-rescue:C-Device
- G1, PlatedHole1: symbol Mechanical:MountingHole -> AGB-E02-20-rescue:MountingHole-Mechanical
- Pad1, Pad2, Pad3, Pad4: symbol Mechanical:MountingHole_Pad -> AGB-E02-20-rescue:MountingHole_Pad-Mechanical
- R1, R2, R3, R4, R5: symbol Device:R -> AGB-E02-20-rescue:R-Device
Changed lines of the file:
@@
 $EndComp
 $Comp
-L power:+3.3V #PWR0101
+L AGB-E02-20-rescue:+3.3V-power #PWR0101
 U 1 1 5DFEEB6D
 P 7500 5875
@@
 CS2
 $Comp
-L power:GND #PWR0102
+L AGB-E02-20-rescue:GND-power #PWR0102
 U 1 1 5DFF0CB2
 P 10600 5875
@@
 A4
 $Comp
-L power:GND #PWR0103
+L AGB-E02-20-rescue:GND-power #PWR0103
 U 1 1 5DFF3745
 P 8275 1900
@@
 $EndComp
 $Comp
-L power:GND #PWR0104
+L AGB-E02-20-rescue:GND-power #PWR0104
 U 1 1 5DFF3B77
 P 10425 2200
@@
 $EndComp
 $Comp
-L Device:R R1
+L AGB-E02-20-rescue:R-Device R1
 U 1 1 5DFF4114
 P 7800 2800
@@
 $EndComp
 $Comp
-L Device:R R2
+L AGB-E02-20-rescue:R-Device R2
 U 1 1 5DFF46E0
 P 7800 2700
@@
 $EndComp
 $Comp
-L Device:R R3
+L AGB-E02-20-rescue:R-Device R3
 U 1 1 5DFF4A79
 P 7800 2600
@@
 	7650 2700 7600 2700
 $Comp
-L power:GND #PWR0105
+L AGB-E02-20-rescue:GND-power #PWR0105
 U 1 1 5E0036EB
 P 7600 2700
@@
 $EndComp
 $Comp
-L power:GND #PWR0106
+L AGB-E02-20-rescue:GND-power #PWR0106
 U 1 1 5DFF2B6E
 P 8275 2300
@@
 $EndComp
 $Comp
-L Device:C C3
+L AGB-E02-20-rescue:C-Device C3
 U 1 1 5E003A9F
 P 7725 1975
@@
 $EndComp
 $Comp
-L power:+3.3V #PWR0107
+L AGB-E02-20-rescue:+3.3V-power #PWR0107
 U 1 1 5DFF3198
 P 8275 2100
@@
 $EndComp
 $Comp
-L power:+3.3V #PWR0108
+L AGB-E02-20-rescue:+3.3V-power #PWR0108
 U 1 1 5E00BACB
 P 7725 2125
@@
 $EndComp
 $Comp
-L power:GND #PWR0109
+L AGB-E02-20-rescue:GND-power #PWR0109
 U 1 1 5E00C145
 P 7725 1825
@@
 $EndComp
 $Comp
-L Device:R R5
+L AGB-E02-20-rescue:R-Device R5
 U 1 1 5E00DE81
 P 6350 850
@@
 $EndComp
 $Comp
-L power:+3.3V #PWR0110
+L AGB-E02-20-rescue:+3.3V-power #PWR0110
 U 1 1 5E00E579
 P 6200 850
@@
 $EndComp
 $Comp
-L power:GND #PWR0111
+L AGB-E02-20-rescue:GND-power #PWR0111
 U 1 1 5E00F04F
 P 6500 850
@@
 $EndComp
 $Comp
-L Device:C C2
+L AGB-E02-20-rescue:C-Device C2
 U 1 1 5E00F60E
 P 6175 1750
@@
 $EndComp
 $Comp
-L Device:C C1
+L AGB-E02-20-rescue:C-Device C1
 U 1 1 5E01A6B1
 P 3600 2275
@@
 $EndComp
 $Comp
-L Device:R R4
+L AGB-E02-20-rescue:R-Device R4
 U 1 1 5E01B00C
 P 3600 3000
@@
 $EndComp
 $Comp
-L power:+3.3V #PWR0112
+L AGB-E02-20-rescue:+3.3V-power #PWR0112
 U 1 1 5E01B83F
 P 3600 3150
@@
 $EndComp
 $Comp
-L power:+3.3V #PWR0113
+L AGB-E02-20-rescue:+3.3V-power #PWR0113
 U 1 1 5E01C361
 P 3600 2125
@@
 $EndComp
 $Comp
-L power:GND #PWR0114
+L AGB-E02-20-rescue:GND-power #PWR0114
 U 1 1 5E01C5C5
 P 3600 2425
@@
 $EndComp
 $Comp
-L power:GND #PWR0115
+L AGB-E02-20-rescue:GND-power #PWR0115
 U 1 1 5E01D863
 P 3600 2850
@@
 $EndComp
 $Comp
-L power:+3.3V #PWR0116
+L AGB-E02-20-rescue:+3.3V-power #PWR0116
 U 1 1 5E01EB01
 P 6175 1900
@@
 $EndComp
 $Comp
-L power:GND #PWR0117
+L AGB-E02-20-rescue:GND-power #PWR0117
 U 1 1 5E01F666
 P 6175 1600
@@
 $EndComp
 $Comp
-L power:GND #PWR0118
+L AGB-E02-20-rescue:GND-power #PWR0118
 U 1 1 5E028389
 P 10500 5875
@@
 $EndComp
 $Comp
-L power:GND #PWR0119
+L AGB-E02-20-rescue:GND-power #PWR0119
 U 1 1 5E039B7F
 P 4450 1300
@@
 $EndComp
 $Comp
-L power:GND #PWR0120
+L AGB-E02-20-rescue:GND-power #PWR0120
 U 1 1 5E03A3E2
 P 4450 2000
@@
 $EndComp
 $Comp
-L power:GND #PWR0121
+L AGB-E02-20-rescue:GND-power #PWR0121
 U 1 1 5E03A8A1
 P 4450 3200
@@
 $EndComp
 $Comp
-L power:GND #PWR0122
+L AGB-E02-20-rescue:GND-power #PWR0122
 U 1 1 5E03AAA3
 P 4450 3300
@@
 $EndComp
 $Comp
-L power:GND #PWR0123
+L AGB-E02-20-rescue:GND-power #PWR0123
 U 1 1 5E03AD00
 P 4450 3400
@@
 $EndComp
 $Comp
-L power:GND #PWR0124
+L AGB-E02-20-rescue:GND-power #PWR0124
 U 1 1 5E03B247
 P 5650 3100
@@
 $EndComp
 $Comp
-L power:GND #PWR0125
+L AGB-E02-20-rescue:GND-power #PWR0125
 U 1 1 5E03B6BD
 P 5650 2100
@@
 $EndComp
 $Comp
-L power:GND #PWR0126
+L AGB-E02-20-rescue:GND-power #PWR0126
 U 1 1 5E03B9C3
 P 5650 1500
@@
 $EndComp
 $Comp
-L power:GND #PWR0127
+L AGB-E02-20-rescue:GND-power #PWR0127
 U 1 1 5E03BABF
 P 5650 1400
@@
 $EndComp
 $Comp
-L power:+3.3V #PWR0128
+L AGB-E02-20-rescue:+3.3V-power #PWR0128
 U 1 1 5E03EB98
 P 5650 2000
@@
 $EndComp
 $Comp
-L power:+3.3V #PWR0129
+L AGB-E02-20-rescue:+3.3V-power #PWR0129
 U 1 1 5E03F059
 P 5650 3200
@@
 $EndComp
 $Comp
-L power:+3.3V #PWR0130
+L AGB-E02-20-rescue:+3.3V-power #PWR0130
 U 1 1 5E03F2A3
 P 5650 3300
@@
 $EndComp
 $Comp
-L power:+3.3V #PWR0131
+L AGB-E02-20-rescue:+3.3V-power #PWR0131
 U 1 1 5E0400DD
 P 4450 2100
@@
 $EndComp
 $Comp
-L power:+3.3V #PWR0132
+L AGB-E02-20-rescue:+3.3V-power #PWR0132
 U 1 1 5E04026A
 P 4450 1500
@@
 $EndComp
 $Comp
-L power:+3.3V #PWR0133
+L AGB-E02-20-rescue:+3.3V-power #PWR0133
 U 1 1 5E04053C
 P 4450 1400
@@
 D7
 $Comp
-L Mechanical:MountingHole PlatedHole1
+L AGB-E02-20-rescue:MountingHole-Mechanical PlatedHole1
 U 1 1 5F1CF176
 P 6675 3625
@@
 $EndComp
 $Comp
-L Mechanical:MountingHole_Pad Pad1
+L AGB-E02-20-rescue:MountingHole_Pad-Mechanical Pad1
 U 1 1 5F1D11A5
 P 6725 4125
@@
 $EndComp
 $Comp
-L Mechanical:MountingHole_Pad Pad2
+L AGB-E02-20-rescue:MountingHole_Pad-Mechanical Pad2
 U 1 1 5F1D1E72
 P 6725 4325
@@
 $EndComp
 $Comp
-L Mechanical:MountingHole_Pad Pad3
+L AGB-E02-20-rescue:MountingHole_Pad-Mechanical Pad3
 U 1 1 5F1D2265
 P 6725 4525
@@
 $EndComp
 $Comp
-L power:GND #PWR0134
+L AGB-E02-20-rescue:GND-power #PWR0134
 U 1 1 5F1D3C86
 P 6625 4125
@@
 $EndComp
 $Comp
-L power:GND #PWR0135
+L AGB-E02-20-rescue:GND-power #PWR0135
 U 1 1 5F1D408B
 P 6625 4325
@@
 $EndComp
 $Comp
-L power:GND #PWR0136
+L AGB-E02-20-rescue:GND-power #PWR0136
 U 1 1 5F1D4442
 P 6625 4525
@@
 $EndComp
 $Comp
-L Mechanical:MountingHole G1
+L AGB-E02-20-rescue:MountingHole-Mechanical G1
 U 1 1 5F1DA8DA
 P 6775 4925
@@
 $EndComp
 $Comp
-L Mechanical:MountingHole_Pad Pad4
+L AGB-E02-20-rescue:MountingHole_Pad-Mechanical Pad4
 U 1 1 5F207589
 P 6725 4725
@@
 $EndComp
 $Comp
-L power:GND #PWR0137
+L AGB-E02-20-rescue:GND-power #PWR0137
 U 1 1 5F20758F
 P 6625 4725
