File: DMG-KFDN-01/DMG-KFDN-01.kicad_sch (KiCad schematic)
At the start: 15 parts, among them U0 CartBus, U1 LH538MNP, U2 MBC3, U3 GM76C256CLLFW70, U4 BA6129AF, X1 Crystal

Commit message: Update DMG-KFDN-01
Parts:
- removed Batt_CR2025: Battery_Cell, NintendoFootprints:CR2025, symbol Device:Battery_Cell
- removed U0: CartBus, NintendoFootprints:CartBus, symbol NintendoSymbols:CartBus
- added BT1: Battery_Cell, Custom:CR2025_Tabbed, symbol Device:Battery_Cell
- added J0: CartBus, HDR_Gameboy_Cartridges:GB_Cartridge_Front_Only, symbol NintendoSymbols:CartBus
- added TP1: RTC_VOUT, Custom:GameBoy_Testpoint, symbol Connector:TestPoint
- added TP2: VBatt, Custom:GameBoy_Testpoint, symbol Connector:TestPoint
- added TP3: BT+, Custom:GameBoy_Testpoint, symbol Connector:TestPoint
- added TP4: GND, Custom:GameBoy_Testpoint, symbol Connector:TestPoint
- added TP5: 3x3, HDR_Gameboy:3x3mm_Pad, symbol Connector:TestPoint
- added TP6: Date Indicator, HDR_Gameboy_Date_Indicators:12 December, symbol Connector:TestPoint
- C1, C2, C3, C4, C5: footprint Capacitor_SMD:C_0603_1608Metric -> Capacitor_SMD:C_0805_2012Metric
- R1, R2, Z1: footprint Resistor_SMD:R_0603_1608Metric -> Resistor_SMD:R_0805_2012Metric
- U3: footprint NintendoFootprints:GM76C256CLLFW70 -> Package_SO:SOIC-28W_7.5x17.9mm_P1.27mm
Connections:
- net +5V: now also J0.1 (VCC)
- net A0: now also J0.6 (A0)
- net A1: now also J0.7 (A1)
- net A10: now also J0.16 (A10)
- net A11: now also J0.17 (A11)
- net A12: now also J0.18 (A12)
- net A13: now also J0.19 (A13)
- net A14: now also J0.20 (A14)
- net A15: now also J0.21 (A15)
- net A2: now also J0.8 (A2)
- net A3: now also J0.9 (A3)
- net A4: now also J0.10 (A4)
- net A5: now also J0.11 (A5)
- net A6: now also J0.12 (A6)
- net A7: now also J0.13 (A7)
- net A8: now also J0.14 (A8)
- net A9: now also J0.15 (A9)
- net Batt: now also TP2.1
- net CLK: now also J0.2 (CLK~{})
- net D0: now also J0.22 (D0)
- net D1: now also J0.23 (D1)
- net D2: now also J0.24 (D2)
- net D3: now also J0.25 (D3)
- net D4: now also J0.26 (D4)
- net D5: now also J0.27 (D5)
- net D6: now also J0.28 (D6)
- net D7: now also J0.29 (D7)
- net GND: now also BT1.2 (-), J0.32 (GND), TP4.1, TP5.1, TP6.1
- net RESET: now also J0.30 (RST)
- net Vout: now also TP1.1
- net WR: now also J0.3 (WR)
- net \RD: now also J0.4 (RD)
- net BT+: now reaches R1.1
- net BT+: now also BT1.1 (+), TP3.1
- net BattCS renamed \RST
Other:
- title: DMG-KFDN-01 -> (none)
